File: Schematics/xymatics-e64.kicad_pcb (KiCad board)
At the start: 2 copper layers, 42 x 42 mm, 270 parts, among them J1 ETHERNET, J10 RPI FAN, J11 RPI-GPIO, J12 STM32 SWD, J13 X-STOP, J14 Y-STOP, J15 Z-STOP, J16 5V POWER, J17 CAN1, J18 CAN2, J19 CAN3, J2 MICRO SD CARD, J20 CAN4, J21 CAN5, J22 CAN6, J23 CAN7, J24 CAN8, J25 FAN1, J26 HOTEND, J27 FAN2, J28 FAN3, J29 FAN4, J3 HDMI, J30 FAN5, J31 CAN IN, J32 HEATBED, J33 FAN1, J34 FAN2, J35 BED THERMISTOR, J36 TEMP, J37 STOP, J4 CAMERA, J41 I2C, J43 SPINDLE/LASER, J44 EXTRUDER, J45 SWD, J5 DISPLAY, J6 MICRO USB, J7 USB_A, J8 USB JST, J9 RPI CONFIG, Q1 HEATBED, Q10 X42 MOSFET, Q2 FAN1, Q3 FAN2, Q4 FAN3, Q5 FAN4, Q6 FAN5, Q7 E0-HEAT, Q8 FAN1, Q9 FAN2, SW1 RPI WAKE, SW2 STM32 RESET, SW3 STM32 BOOT, SW4 EN, SW5 BOOT, U1 RPI-CM4, U10 STM32F407VET6, U11 MOTOR A, U12 MOTOR B, U13 MOTOR Z1, U14 MOTOR Z2, U15 MOTOR Z3, U16 TPS54302, U17 AMS1117CD-3.3, U18 TJA1051T-3, U19 SSD1306-0.91, U2 TPS2065CDBV, U20 STM32G0B1CBTx, U21 TJA1051T-3, U22 74LVC1G17, U23 TPS54302, U24 AMS1117CD-3.3, U26 ADXL345BCCZ, U27 74LVC1G17, U28 74LVC1G17, U29 TMC2209-LA-T, U3 TPS2065CDBV, U4 CH334R, U5 FSUSB42MUX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

Commit message: Update X42 schematics, Update X42 PCB
Removed X42 Endstops (re-add in next revision)
Parts:
- removed J37: STOP, Connector_JST:JST_XH_B3B-XH-A_1x03_P2.50mm_Vertical
- removed R58: 10K, Resistor_SMD:R_0805_2012Metric
- C57, C58, C59, C72, C73, C76, C77, C82, C83, C84, L4, Q10, R42, R63, R64, R65, R66, R67, R68, R69, R70, R75, R77, R79, U26, U27, Y3: moved to B.Cu
- J41: footprint Connector_JST:JST_XH_B4B-XH-A_1x04_P2.50mm_Vertical -> Connector_PinHeader_2.54mm:PinHeader_1x04_P2.54mm_Vertical_SMD_Pin1Right
- J43: footprint Connector_JST:JST_XH_B2B-XH-A_1x02_P2.50mm_Vertical -> Connector_PinHeader_2.54mm:PinHeader_1x02_P2.54mm_Vertical_SMD_Pin1Right
- moved U27 143.6 mm to (59.5, 175.5)
- moved R47 137.1 mm to (39.3, 188.3)
- moved R42 136.4 mm to (53.0, 172.5), turned to 180 degrees
- moved Q10 135.8 mm to (58.2, 185.8)
- moved J43 132.2 mm to (33.6, 174.3)
- moved R69 130.3 mm to (63.5, 174.6), turned to 180 degrees
- moved R70 129.7 mm to (63.5, 176.5)
- moved C77 127.3 mm to (68.0, 181.0)
- moved R78 125.8 mm to (53.9, 185.6), turned to 90 degrees
- moved R75 125.0 mm to (60.2, 167.5), turned to -90 degrees
- moved R46 124.0 mm to (39.3, 182.0)
- moved R67 122.9 mm to (53.7, 169.9), turned to 180 degrees
- moved R64 118.8 mm to (53.2, 154.6), turned to 180 degrees
- moved C59 118.8 mm to (50.6, 176.1)
- moved C76 116.6 mm to (59.5, 170.5), turned to 180 degrees
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Connections:
- C56 pad 2: GND -> XGND
- C57 pad 1: GND -> XGND
- C58 pad 1: GND -> XGND
- C59 pad 2: GND -> XGND
- C61 pad 1: GND -> XGND
- C62 pad 2: GND -> XGND
- C63 pad 2: GND -> XGND
- C64 pad 2: GND -> XGND
- C67 pad 2: GND -> XGND
- C68 pad 2: GND -> XGND
- C69 pad 2: GND -> XGND
- C70 pad 2: GND -> XGND
- C72 pad 2: GND -> XGND
- C73 pad 2: GND -> XGND
- C75 pad 1: GND -> XGND
- C77 pad 1: GND -> XGND
- C78 pad 1: GND -> XGND
- C79 pad 1: GND -> XGND
- C80 pad 2: GND -> XGND
- C82 pad 2: GND -> XGND
- C83 pad 2: GND -> XGND
- C84 pad 2: GND -> XGND
- D13 pad 1: GND -> XGND
- D16 pad 1: GND -> XGND
- D17 pad 1: GND -> XGND
- H1 pad 1: GND -> XGND
- H2 pad 1: GND -> XGND
- J31 pad 1: GND -> XGND
- J36 pad 2: GND -> XGND
- J41 pad 2: GND -> XGND
- J45 pad 1: GND -> XGND
- L4 pad 1: /X42/X42-3V3 -> /X42/3V3
- Q10 pad 3: GND -> XGND
- Q7 pad 4: GND -> XGND
- Q8 pad 3: GND -> XGND
- Q9 pad 3: GND -> XGND
- R42 pad 1: GND -> XGND
- R43 pad 2: GND -> XGND
- R44 pad 1: GND -> XGND
- R55 pad 1: GND -> XGND
- R57 pad 1: GND -> XGND
- R68 pad 2: GND -> XGND
- R69 pad 1: GND -> XGND
- R73 pad 2: GND -> XGND
- R74 pad 2: GND -> XGND
- R78 pad 1: GND -> XGND
- SW4 pad 1: GND -> XGND
- SW5 pad 1: GND -> XGND
- U20 pad 42: unconnected-(U20-PB3-Pad42) -> /X42/X42-SCL
- U20 pad 43: unconnected-(U20-PB4-Pad43) -> /X42/X42-SDA
- U20 pad 44: /X42/X42-ENDSTOP -> unconnected-(U20-PB5-Pad44)
- U20 pad 7: GND -> XGND
- U21 pad 2: GND -> XGND
- U21 pad 8: GND -> XGND
- U22 pad 2: GND -> XGND
- U22 pad 3: GND -> XGND
- U23 pad 1: GND -> XGND
- U24 pad 1: GND -> XGND
- U26 pad 11: GND -> XGND
- U26 pad 2: GND -> XGND
- U26 pad 4: GND -> XGND
- U26 pad 5: GND -> XGND
- U27 pad 2: GND -> XGND
- U27 pad 3: GND -> XGND
- U29 pad 10: GND -> XGND
- U29 pad 13: GND -> XGND
- U29 pad 18: GND -> XGND
- U29 pad 20: GND -> XGND
- U29 pad 29: GND -> XGND
- U29 pad 3: GND -> XGND
- U29 pad 7: GND -> XGND
- U29 pad 9: GND -> XGND
- Y3 pad 2: GND -> XGND
- Y3 pad 4: GND -> XGND
Routing:
- net /X42/3V3: track 78.2 -> 172.5 mm, vias 5 -> 12
- net XGND: track 0.00 -> 69.4 mm
- net /X42/24V: track 58.6 -> 109.0 mm, vias 4 -> 8
- net GND: track 45.2 -> 0.00 mm
- net /X42/X42-3V3: track 0.00 -> 43.6 mm, vias 0 -> 1
- net /X42/X42-CS: track 0.00 -> 33.1 mm, vias 0 -> 5
- net /X42/X42-FAN2: track 0.00 -> 31.2 mm, vias 0 -> 4
- net Net-(D14-A): track 0.00 -> 31.1 mm, vias 0 -> 3
- net /X42/X42-MOSI: track 0.00 -> 27.5 mm, vias 0 -> 1
- net /X42/5V: track 79.9 -> 107.3 mm, vias 2 -> 4
- net Net-(U20-PF1): track 0.00 -> 25.8 mm, vias 0 -> 1
- net /X42/X42-FAN1: track 0.00 -> 25.2 mm, vias 0 -> 4
- net Net-(U20-PF0): track 0.00 -> 24.0 mm, vias 0 -> 5
- net /X42/X42-SCL: track 0.00 -> 23.6 mm, vias 0 -> 2
- net /X42/X42-CLK: track 0.00 -> 23.3 mm, vias 0 -> 3
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
Commit message: Update E64 schematics
Finish E64 PCB
Parts:
- removed R36, R37: 4.7K, Resistor_SMD:R_0805_2012Metric
- removed Y1: 24MHZ, Crystal:Crystal_HC49-4H_Vertical
- added C71: 100NF, Capacitor_SMD:C_0805_2012Metric, F.Cu at (67.7, 67.4)
- added C81: 100NF, Capacitor_SMD:C_0805_2012Metric, F.Cu at (67.7, 60.9)
- added C85: 4.7UF, Capacitor_SMD:C_0805_2012Metric, F.Cu at (67.7, 63.0)
- added C86: 100NF, Capacitor_SMD:C_0805_2012Metric, F.Cu at (67.7, 65.2)
- added C87: 100NF, Capacitor_SMD:C_0805_2012Metric, F.Cu at (67.7, 69.6)
- added D15: 20A, Diode_SMD:D_SMB, F.Cu at (73.2, 62.2)
- added F1: 10A, Fuse:Fuse_Blade_ATO_directSolder, F.Cu at (60.9, 56.4)
- added H3: MountingHole_Pad, MountingHole:MountingHole_3mm_Pad, F.Cu at (59.0, 30.2)
- added H4: MountingHole_Pad, MountingHole:MountingHole_3mm_Pad, F.Cu at (242.0, 30.0)
- added H5: MountingHole_Pad, MountingHole:MountingHole_3mm_Pad, F.Cu at (58.8, 119.8)
- added J37: 24V IN, TerminalBlock:TerminalBlock_MaiXu_MX126-5.0-02P_1x02_P5.00mm, F.Cu at (59.6, 63.4)
- added J38: MOTOR A, Connector_JST:JST_XH_B4B-XH-A_1x04_P2.50mm_Vertical, F.Cu at (70.4, 29.5)
- added J39: MOTOR B, Connector_JST:JST_XH_B4B-XH-A_1x04_P2.50mm_Vertical, F.Cu at (91.6, 29.5)
- added J40: MOTOR Z1, Connector_JST:JST_XH_B4B-XH-A_1x04_P2.50mm_Vertical, F.Cu at (112.8, 29.5)
- added J42: MOTOR Z2, Connector_JST:JST_XH_B4B-XH-A_1x04_P2.50mm_Vertical, F.Cu at (134.0, 29.5)
- added J46: MOTOR Z3, Connector_JST:JST_XH_B4B-XH-A_1x04_P2.50mm_Vertical, F.Cu at (155.3, 29.5)
- added Y4: 24MHZ, Crystal:Crystal_SMD_Abracon_ABM3B-4Pin_5.0x3.2mm, F.Cu at (231.6, 67.2)
- D18: value STM32 POWER -> POWER
- D19: value STM32 STATUS -> STATUS
- D4: value B340 -> 20A; footprint Diode_SMD:D_SMC -> Diode_SMD:D_SMB
- D5, D6, D7, D8, D9: value B340 -> 1N5819WS; footprint Diode_SMD:D_SMC -> Diode_SMD:D_SOD-323
- J32: footprint Connector_JST:JST_XH_B2B-XH-A_1x02_P2.50mm_Vertical -> TerminalBlock:TerminalBlock_MaiXu_MX126-5.0-02P_1x02_P5.00mm
- R24: footprint Resistor_SMD:R_0805_2012Metric -> Resistor_SMD:R_1206_3216Metric
- SW2: value STM32 RESET -> RESET
- SW3: value STM32 BOOT -> BOOT
- U17: footprint Package_TO_SOT_SMD:TO-252-3_TabPin2 -> Package_TO_SOT_SMD:TO-252-2
- moved J25 335.0 mm to (154.5, 68.8), turned to 180 degrees
- moved J27 334.9 mm to (154.5, 75.8), turned to 180 degrees
- moved J28 334.8 mm to (154.5, 82.8), turned to 180 degrees
- moved J29 334.7 mm to (154.5, 89.8), turned to 180 degrees
- moved J30 334.6 mm to (154.5, 96.8), turned to 180 degrees
- moved J2 323.2 mm to (239.8, 46.2), turned to -90 degrees
- moved J24 320.5 mm to (157.9, 117.5), turned to 180 degrees
- moved J23 312.0 mm to (146.6, 117.5), turned to 180 degrees
- moved J22 304.1 mm to (135.2, 117.5), turned to 180 degrees
- moved J21 294.8 mm to (123.8, 117.5), turned to 180 degrees
- moved C39 293.8 mm to (167.8, 32.4), turned to 180 degrees
- moved D5 291.2 mm to (147.2, 70.0), turned to 180 degrees
- moved D6 291.2 mm to (147.2, 77.0), turned to 180 degrees
- moved D7 291.1 mm to (147.2, 84.0), turned to 180 degrees
- moved D8 291.0 mm to (147.2, 91.0), turned to 180 degrees
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Connections:
- D4 pad 2: Net-(D4-A) -> Net-(D15-K)
- H1 pad 1: XGND -> unconnected-(H1-Pad1)
- H2 pad 1: XGND -> unconnected-(H2-Pad1)
- J16 pad 3: /USB_5V -> USB_5V
- J32 pad 2: Net-(D4-A) -> Net-(J32-Pin_2)
- J6 pad 1: /RPI-CM4/USB_5V -> USB_5V
- Q1 pad 1: Net-(D4-A) -> Net-(Q1-G)
- Q1 pad 2: Net-(Q1-G) -> Net-(J32-Pin_2)
- R14 pad 1: Net-(U10-PB11) -> Net-(U10-PD7)
- R15 pad 1: Net-(U10-PB12) -> Net-(U10-PD6)
- R16 pad 1: Net-(U10-PB13) -> Net-(U10-PD5)
- R17 pad 1: Net-(U10-PB14) -> Net-(U10-PD4)
- R18 pad 1: Net-(U10-PB15) -> Net-(U10-PD3)
- U10 pad 48: Net-(U10-PB11) -> unconnected-(U10-PB11-Pad48)
- U10 pad 51: Net-(U10-PB12) -> unconnected-(U10-PB12-Pad51)
- U10 pad 52: Net-(U10-PB13) -> unconnected-(U10-PB13-Pad52)
- U10 pad 53: Net-(U10-PB14) -> unconnected-(U10-PB14-Pad53)
- U10 pad 54: Net-(U10-PB15) -> unconnected-(U10-PB15-Pad54)
- U10 pad 70: /STM32_USB- -> STM32_USB-
- U10 pad 71: /STM32_USB+ -> STM32_USB+
- U10 pad 84: unconnected-(U10-PD3-Pad84) -> Net-(U10-PD3)
- U10 pad 85: unconnected-(U10-PD4-Pad85) -> Net-(U10-PD4)
- U10 pad 86: unconnected-(U10-PD5-Pad86) -> Net-(U10-PD5)
- U10 pad 87: unconnected-(U10-PD6-Pad87) -> Net-(U10-PD6)
- U10 pad 88: unconnected-(U10-PD7-Pad88) -> Net-(U10-PD7)
- U10 pad 95: Net-(U10-PB8) -> unconnected-(U10-PB8-Pad95)
- U10 pad 96: Net-(U10-PB9) -> unconnected-(U10-PB9-Pad96)
- U4 pad 7: /RPI-CM4/STM32_USB- -> STM32_USB-
- U4 pad 8: /RPI-CM4/STM32_USB+ -> STM32_USB+
Routing:
- net +24V: track 0.00 -> 514.4 mm, vias 0 -> 2
- net +3V3: track 0.00 -> 428.6 mm, vias 0 -> 14
- net +5V: track 0.00 -> 417.3 mm, vias 0 -> 10
- net +3.3V: track 0.00 -> 275.2 mm, vias 0 -> 7
- net USB_5V: track 0.00 -> 231.7 mm, vias 0 -> 2
- net GND: track 0.00 -> 214.2 mm, vias 0 -> 8
- net /RPI-CM4/RPI_SCL: track 0.00 -> 190.1 mm, vias 0 -> 6
- net /RPI-CM4/RPI_SDA: track 0.00 -> 189.9 mm, vias 0 -> 6
- net STM32_USB-: track 0.00 -> 179.9 mm, vias 0 -> 2
- net STM32_USB+: track 0.00 -> 179.2 mm, vias 0 -> 2
- net Net-(J17-Pin_3): track 0.00 -> 116.6 mm
- net Net-(J17-Pin_4): track 0.00 -> 114.4 mm
- net Net-(U10-PD7): track 0.00 -> 83.3 mm
- net /MOTOR5_DIR: track 0.00 -> 83.1 mm, vias 0 -> 1
- net /MOTOR5_STEP: track 0.00 -> 80.9 mm, vias 0 -> 1
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- added copper zone on B.Cu, net GND
- added copper zone on F.Cu, net GND
- added copper zone on B.Cu, net XGND
- added copper zone on F.Cu, net XGND
Other:
- board size 42 x 42 mm -> 191.2 x 164 mm
- board text added: "REV0"
- board text added: "XYMATICS E64"
